File: LEDS.kicad_sch (KiCad schematic)
At the start: 0 parts

Commit message: added manufacturing files
Parts:
- added D10, D11, D12, D13, D14, D15, D16, D17, D18, D19, D20, D21, D22, D23, D24, D25, D26, D27, D28, D29, D5, D6, D7, D8, D9: LED, Custom:LED-ThroughHole-And-SMD0805, symbol Device:LED
- added JP1: SolderJumper_3_Bridged12, Jumper:SolderJumper-3_P1.3mm_Bridged12_RoundedPad1.0x1.5mm, symbol Jumper:SolderJumper_3_Bridged12
- added R10 (x5): 0603, Resistor_SMD:R_0603_1608Metric, symbol Device:R
- added R10 (x5): 0805, Resistor_SMD:R_0805_2012Metric, symbol Device:R
Connections:
- new net: D20.2 (A), D22.2 (A), D24.2 (A), D26.2 (A), D28.2 (A), R10.2, R10.2
- new net: D15.2 (A), D16.2 (A), D17.2 (A), D18.2 (A), D19.2 (A), R10.2, R10.2
- new net: D10.2 (A), D11.2 (A), D12.2 (A), D13.2 (A), D14.2 (A), R10.2, R10.2
- new net: D21.2 (A), D23.2 (A), D25.2 (A), D27.2 (A), D29.2 (A), R10.2, R10.2
- new net: D5.2 (A), D6.2 (A), D7.2 (A), D8.2 (A), D9.2 (A), R10.2, R10.2
- new net +5V: JP1.1 (A)
- new net +VSW: JP1.2 (C), R10.1, R10.1, R10.1, R10.1, R10.1, R10.1, R10.1, R10.1, R10.1, R10.1
- new net GND: D10.1 (K), D11.1 (K), D12.1 (K), D13.1 (K), D14.1 (K), D15.1 (K), D16.1 (K), D17.1 (K), D18.1 (K), D19.1 (K), D20.1 (K), D21.1 (K), D22.1 (K), D23.1 (K), D24.1 (K), D25.1 (K), D26.1 (K), D27.1 (K), D28.1 (K), D29.1 (K), D5.1 (K), D6.1 (K), D7.1 (K), D8.1 (K), D9.1 (K)
- new net VCC: JP1.3 (B)
